File: Circuits/Transformer Breakout/Transformer Breakout - Parallel.kicad_pcb (KiCad board)
At the start: 2 copper layers, 17.8 x 30.5 mm, 65 parts, among them P1 XFRMR, P2 BRK

Commit message: Circuits: Small updates to Transformer Breakouts: circle icon, removing thermal rings
Parts:
- ? (x63): footprint Footprints:Thermal_Via -> Footprints:Thermal_Via_NoRing
