File: Circuits/3rd Order Butterworth LPAD/LPAD.sch (KiCad schematic (older format))
At the start: 24 parts, among them P1 INPUT, P2 TWEETER, P3 WOOFER_A, P4 WOOFER_B, SW1 Attenuation, SW2 Phase, SW3 Attenuation, SW4 Phase, SW5 Bypass, SW6 Phase

Commit message: Circuits: Updating X+ - reducing via count, updating resistor footprints
Parts:
- R99: footprint Resistors_ThroughHole:Resistor_Horizontal_RM10mm -> (none)
Connections:
- net Bypass: now reaches SW4.1 (A), SW4.6 (C), SW5.2
- net Low_Attenuated: now reaches SW3.2 (B), SW3.5 (B), SW4.3 (C), SW4.4 (A)
- net High_Attenuated: now reaches SW1.2 (B), SW1.5 (B), SW2.1 (A), SW2.6 (C)
- net Low_Secondary: now reaches SW5.1, SW6.3 (C), SW6.4 (A)
- net High: now reaches C3.2, C4.2, R1.2, SW1.1 (A)
- net Low: now reaches L3.1, R3.2, SW3.1 (A)
- net High_Shunt: now reaches R2.2, SW1.6 (C)
- net Low_Shunt: now reaches R4.2, SW3.6 (C)
- net High_Xover: now reaches C1.2, C2.2, C3.1, C4.1, L1.1
- net Low_Xover: now reaches C5.1, C6.1, L2.1, L3.2
Other:
- note added: "24Ω Nominal"
- note removed: "20Ω Nominal"
Changed lines of the file:
@@
 P 5800 1200
 F 0 "R1" V 5880 1200 50  0000 C CNN
-F 1 "2Ω" V 5800 1200 50  0000 C CNN
+F 1 "2Ω" V 5800 1200 39  0000 C CNN
 F 2 "Footprints:R_WIREWOUND_25W" V 5730 1200 30  0001 C CNN
 F 3 "" H 5800 1200 30  0000 C CNN
@@
 P 5800 2300
 F 0 "R2" V 5880 2300 50  0000 C CNN
-F 1 "25Ω" V 5800 2300 50  0000 C CNN
+F 1 "25Ω" V 5800 2300 39  0000 C CNN
 F 2 "Footprints:R_WIREWOUND_25W" V 5730 2300 30  0001 C CNN
 F 3 "" H 5800 2300 30  0000 C CNN
@@
 P 5800 3950
 F 0 "R3" V 5880 3950 50  0000 C CNN
-F 1 "2Ω" V 5800 3950 50  0000 C CNN
+F 1 "2Ω" V 5800 3950 39  0000 C CNN
 F 2 "Footprints:R_WIREWOUND_100W" V 5730 3950 30  0001 C CNN
 F 3 "" H 5800 3950 30  0000 C CNN
@@
 P 5800 5300
 F 0 "R4" V 5880 5300 50  0000 C CNN
-F 1 "24Ω" V 5800 5300 50  0000 C CNN
+F 1 "24Ω" V 5800 5300 43  0000 C CNN
 F 2 "Footprints:R_WIREWOUND_100W" V 5730 5300 30  0001 C CNN
 F 3 "" H 5800 5300 30  0000 C CNN
@@
 15.6 μF Actual\n
 Text Notes 5950 5300 0    60   ~ 0
-20Ω Nominal
+24Ω Nominal
 Text Notes 5950 5400 0    60   ~ 0
 24Ω Actual
 Text Notes 5900 2300 0    60   ~ 0
-20Ω Nominal
+24Ω Nominal
 Text Notes 5900 2400 0    60   ~ 0
 25Ω Actual
@@
 F 0 "R99" V 3400 7100 50  0000 C CNN
 F 1 "DUMMY" V 3500 7100 50  0000 C CNN
-F 2 "Resistors_ThroughHole:Resistor_Horizontal_RM10mm" V 3330 7100 30  0000 C CNN
+F 2 "" V 3330 7100 30  0000 C CNN
 F 3 "" H 3400 7100 30  0000 C CNN
 	1    3400 7100
@@
 Wire Wire Line
 	3650 7100 3550 7100
+Text Label 4850 3850 0    39   ~ 0
+Low
+Text Label 7100 3850 0    39   ~ 0
+Low_Attenuated
+Text Label 7200 5250 0    39   ~ 0
+Bypass
+Text Label 4850 1100 0    39   ~ 0
+High
+Text Label 7250 1100 0    39   ~ 0
+High_Attenuated
+Text Label 8100 5550 1    39   ~ 0
+Low_Secondary
+Text Label 3850 4500 1    39   ~ 0
+Low_Xover
+Text Label 3850 1650 1    39   ~ 0
+High_Xover
+Text Label 5800 5000 1    39   ~ 0
+Low_Shunt
+Text Label 5800 2150 1    39   ~ 0
+High_Shunt
 $EndSCHEMATC
