File: Circuits/AAA Cap Board/AAA Cap Board.sch (KiCad schematic (older format))
At the start: 18 parts

Commit message: AAA Cap Board: Edits?
Parts:
- C1, C10, C14, C15, C8, C9: symbol C -> C-RESCUE-AAA_Cap_Board
- C11, C12, C13, C2: symbol CP -> CP-RESCUE-AAA_Cap_Board
- C3, C4, C5, C6, C7: symbol CP1 -> CP1-RESCUE-AAA_Cap_Board
Changed lines of the file:
@@
 EESchema Schematic File Version 2
+LIBS:AAA Cap Board-rescue
 LIBS:power
 LIBS:device
@@
 LIBS:w_device
 LIBS:aaa_terminal
+LIBS:AAA Cap Board-cache
 EELAYER 25 0
 EELAYER END
@@
 $EndDescr
 $Comp
-L C C14
+L C-RESCUE-AAA_Cap_Board C14
 U 1 1 564FE5D4
 P 8400 3100
@@
 $EndComp
 $Comp
-L C C10
+L C-RESCUE-AAA_Cap_Board C10
 U 1 1 564FE638
 P 6600 3100
@@
 $EndComp
 $Comp
-L C C9
+L C-RESCUE-AAA_Cap_Board C9
 U 1 1 564FE656
 P 6150 3100
@@
 $EndComp
 $Comp
-L C C8
+L C-RESCUE-AAA_Cap_Board C8
 U 1 1 564FE68D
 P 5700 3100
@@
 $EndComp
 $Comp
-L C C1
+L C-RESCUE-AAA_Cap_Board C1
 U 1 1 564FE6D1
 P 2600 3100
@@
 $EndComp
 $Comp
-L CP C13
+L CP-RESCUE-AAA_Cap_Board C13
 U 1 1 564FE760
 P 7950 3100
@@
 $EndComp
 $Comp
-L CP C12
+L CP-RESCUE-AAA_Cap_Board C12
 U 1 1 564FE7BD
 P 7500 3100
@@
 $EndComp
 $Comp
-L CP C11
+L CP-RESCUE-AAA_Cap_Board C11
 U 1 1 564FE7FB
 P 7050 3100
@@
 $EndComp
 $Comp
-L CP C2
+L CP-RESCUE-AAA_Cap_Board C2
 U 1 1 564FE84F
 P 3050 3100
@@
 $EndComp
 $Comp
-L CP1 C7
+L CP1-RESCUE-AAA_Cap_Board C7
 U 1 1 564FE885
 P 5250 3100
@@
 $EndComp
 $Comp
-L CP1 C6
+L CP1-RESCUE-AAA_Cap_Board C6
 U 1 1 564FE918
 P 4800 3100
@@
 $EndComp
 $Comp
-L CP1 C5
+L CP1-RESCUE-AAA_Cap_Board C5
 U 1 1 564FE973
 P 4350 3100
@@
 $EndComp
 $Comp
-L CP1 C4
+L CP1-RESCUE-AAA_Cap_Board C4
 U 1 1 564FE9BB
 P 3950 3100
@@
 $EndComp
 $Comp
-L CP1 C3
+L CP1-RESCUE-AAA_Cap_Board C3
 U 1 1 564FE9FA
 P 3500 3100
@@
 $EndComp
 $Comp
-L C C15
+L C-RESCUE-AAA_Cap_Board C15
 U 1 1 564FEF54
 P 8850 3100
