File: Circuits/Garage Assistant/Garage Assistant.sch (KiCad schematic (older format))
At the start: 31 parts, among them P1 MOTION_A, P2 MOTION_B, P3 AC_IN, P4 3.5mm_11pin, P5 OUT_A, P6 OUT_B, Q1 TIP122, Q2 TIP122, U1 HiLink_5V3W

Commit message: Circuits: Updated 3d models on Garage Assistant
Parts:
- added R4, R5: 1kΩ, Resistors_ThroughHole:Resistor_Horizontal_RM10mm, symbol R
- D5, D6: value 1N4002 -> 1N4007
- Q1, Q2: value TIP122 -> TIP102
- renumbered R4 to R6, R5 to R7, R6 to R8
Connections:
- net A_RELAY: now also R4.2; no longer Q1.1 (B)
- net B_RELAY: now also R5.2; no longer Q2.1 (B)
- new net: Q2.1 (B), R5.1
- new net: Q1.1 (B), R4.1
Changed lines of the file:
@@
 LIBS:contrib
 LIBS:valves
-LIBS:red_bear_labs
 LIBS:ehryk
 LIBS:w_relay
@@
 Connection ~ 8700 3700
 $Comp
-L GND #PWR01
+L GND #PWR10
 U 1 1 583CF72C
 P 5450 1400
-F 0 "#PWR01" H 5450 1400 30  0001 C CNN
+F 0 "#PWR10" H 5450 1400 30  0001 C CNN
 F 1 "GND" H 5450 1330 30  0001 C CNN
 F 2 "" H 5450 1400 60  0001 C CNN
@@
 $EndComp
 $Comp
-L GND #PWR02
+L GND #PWR9
 U 1 1 583CF78F
 P 3650 4600
-F 0 "#PWR02" H 3650 4600 30  0001 C CNN
+F 0 "#PWR9" H 3650 4600 30  0001 C CNN
 F 1 "GND" H 3650 4530 30  0001 C CNN
 F 2 "" H 3650 4600 60  0001 C CNN
@@
 $EndComp
 $Comp
-L GND #PWR03
+L GND #PWR12
 U 1 1 583CF8CC
 P 5550 4600
-F 0 "#PWR03" H 5550 4600 30  0001 C CNN
+F 0 "#PWR12" H 5550 4600 30  0001 C CNN
 F 1 "GND" H 5550 4530 30  0001 C CNN
 F 2 "" H 5550 4600 60  0001 C CNN
@@
 	5550 4400 5450 4400
 $Comp
-L GND #PWR04
+L GND #PWR20
 U 1 1 583CFAB3
 P 10950 4550
-F 0 "#PWR04" H 10950 4550 30  0001 C CNN
+F 0 "#PWR20" H 10950 4550 30  0001 C CNN
 F 1 "GND" H 10950 4480 30  0001 C CNN
 F 2 "" H 10950 4550 60  0001 C CNN
@@
 $EndComp
 $Comp
-L GND #PWR05
+L GND #PWR16
 U 1 1 583CFB1F
 P 8250 2300
-F 0 "#PWR05" H 8250 2300 30  0001 C CNN
+F 0 "#PWR16" H 8250 2300 30  0001 C CNN
 F 1 "GND" H 8250 2230 30  0001 C CNN
 F 2 "" H 8250 2300 60  0001 C CNN
@@
 $EndComp
 $Comp
-L GND #PWR06
+L GND #PWR18
 U 1 1 583D07E1
 P 9750 5900
-F 0 "#PWR06" H 9750 5900 30  0001 C CNN
+F 0 "#PWR18" H 9750 5900 30  0001 C CNN
 F 1 "GND" H 9750 5830 30  0001 C CNN
 F 2 "" H 9750 5900 60  0001 C CNN
@@
 $EndComp
 $Comp
-L R R4
+L R R6
 U 1 1 583D0879
 P 8950 5800
-F 0 "R4" V 8850 5800 50  0000 C CNN
-F 1 "220Ω" V 8950 5800 50  0000 C CNN
+F 0 "R6" V 8850 5800 50  0000 C CNN
+F 1 "220Ω" V 8950 5800 47  0000 C CNN
 F 2 "Resistors_ThroughHole:Resistor_Horizontal_RM7mm" V 8880 5800 30  0001 C CNN
 F 3 "" H 8950 5800 30  0000 C CNN
@@
 $EndComp
 $Comp
-L GND #PWR07
+L GND #PWR8
 U 1 1 583D111F
 P 3300 4600
-F 0 "#PWR07" H 3300 4600 30  0001 C CNN
+F 0 "#PWR8" H 3300 4600 30  0001 C CNN
 F 1 "GND" H 3300 4530 30  0001 C CNN
 F 2 "" H 3300 4600 60  0001 C CNN
@@
 	10950 4450 10950 4550
 $Comp
-L R R6
+L R R8
 U 1 1 583D1E02
 P 10150 4450
-F 0 "R6" V 10050 4450 50  0000 C CNN
-F 1 "220Ω" V 10150 4450 50  0000 C CNN
+F 0 "R8" V 10050 4450 50  0000 C CNN
+F 1 "220Ω" V 10150 4450 47  0000 C CNN
 F 2 "Resistors_ThroughHole:Resistor_Horizontal_RM7mm" V 10080 4450 30  0001 C CNN
 F 3 "" H 10150 4450 30  0000 C CNN
@@
 P 8150 4200
 F 0 "Q2" H 8400 4275 50  0000 L CNN
-F 1 "TIP122" H 8400 4200 50  0000 L CNN
+F 1 "TIP102" H 8400 4200 50  0000 L CNN
 F 2 "Power_Integrations:TO-220" H 6850 3950 50  0001 L CIN
 F 3 "" H 8150 4200 50  0000 L CNN
@@
 	8250 3900 8250 4000
 $Comp
-L GND #PWR08
+L GND #PWR17
 U 1 1 583D2383
 P 8250 4550
-F 0 "#PWR08" H 8250 4550 30  0001 C CNN
+F 0 "#PWR17" H 8250 4550 30  0001 C CNN
 F 1 "GND" H 8250 4480 30  0001 C CNN
 F 2 "" H 8250 4550 60  0001 C CNN
@@
 P 8150 1950
 F 0 "Q1" H 8400 2025 50  0000 L CNN
-F 1 "TIP122" H 8400 1950 50  0000 L CNN
+F 1 "TIP102" H 8400 1950 50  0000 L CNN
 F 2 "Power_Integrations:TO-220" H 8400 1875 50  0001 L CIN
 F 3 "" H 8150 1950 50  0000 L CNN
@@
 	8250 2150 8250 2300
 $Comp
-L GND #PWR09
+L GND #PWR19
 U 1 1 583D33AB
 P 10950 2300
-F 0 "#PWR09" H 10950 2300 30  0001 C CNN
+F 0 "#PWR19" H 10950 2300 30  0001 C CNN
 F 1 "GND" H 10950 2230 30  0001 C CNN
 F 2 "" H 10950 2300 60  0001 C CNN
@@
 	10950 2200 10950 2300
 $Comp
-L R R5
+L R R7
 U 1 1 583D33B9
 P 10150 2200
-F 0 "R5" V 10050 2200 50  0000 C CNN
-F 1 "220Ω" V 10150 2200 50  0000 C CNN
+F 0 "R7" V 10050 2200 50  0000 C CNN
+F 1 "220Ω" V 10150 2200 47  0000 C CNN
 F 2 "Resistors_ThroughHole:Resistor_Horizontal_RM7mm" V 10080 2200 30  0001 C CNN
 F 3 "" H 10150 2200 30  0000 C CNN
@@
 Text GLabel 9850 2200 0    47   Input ~ 0
 A_LED
-Text GLabel 7800 1950 0    47   Input ~ 0
+Text GLabel 7350 1950 0    47   Input ~ 0
 A_RELAY
-Text GLabel 7800 4200 0    47   Input ~ 0
+Text GLabel 7350 4200 0    47   Input ~ 0
 B_RELAY
 Text GLabel 9850 4450 0    47   Input ~ 0
@@
 CS_CONNECT
 $Comp
-L GND #PWR010
+L GND #PWR6
 U 1 1 583EC6C1
 P 2050 7100
-F 0 "#PWR010" H 2050 7100 30  0001 C CNN
+F 0 "#PWR6" H 2050 7100 30  0001 C CNN
 F 1 "GND" H 2050 7030 30  0001 C CNN
 F 2 "" H 2050 7100 60  0001 C CNN
@@
 NoConn ~ 5450 3500
 $Comp
-L +5V #PWR011
+L +5V #PWR11
 U 1 1 583ECC31
 P 5450 1600
-F 0 "#PWR011" H 5450 1690 20  0001 C CNN
+F 0 "#PWR11" H 5450 1690 20  0001 C CNN
 F 1 "+5V" H 5450 1690 30  0000 C CNN
 F 2 "" H 5450 1600 60  0001 C CNN
@@
 $EndComp
 $Comp
-L GND #PWR012
+L GND #PWR15
 U 1 1 583EEB39
 P 5800 6950
-F 0 "#PWR012" H 5800 6950 30  0001 C CNN
+F 0 "#PWR15" H 5800 6950 30  0001 C CNN
 F 1 "GND" H 5800 6880 30  0001 C CNN
 F 2 "" H 5800 6950 60  0001 C CNN
@@
 	5450 1650 5300 1650
 $Comp
-L +5V #PWR013
+L +5V #PWR7
 U 1 1 583F0557
 P 3000 4100
-F 0 "#PWR013" H 3000 4190 20  0001 C CNN
+F 0 "#PWR7" H 3000 4190 20  0001 C CNN
 F 1 "+5V" H 3000 4190 30  0000 C CNN
 F 2 "" H 3000 4100 60  0001 C CNN
@@
 $EndComp
 $Comp
-L +5V #PWR014
+L +5V #PWR1
 U 1 1 583F4CE6
 P 1600 3150
-F 0 "#PWR014" H 1600 3240 20  0001 C CNN
+F 0 "#PWR1" H 1600 3240 20  0001 C CNN
 F 1 "+5V" H 1600 3240 30  0000 C CNN
 F 2 "" H 1600 3150 60  0001 C CNN
@@
 $EndComp
 $Comp
-L +5V #PWR015
+L +5V #PWR3
 U 1 1 583F4D48
 P 1600 4150
-F 0 "#PWR015" H 1600 4240 20  0001 C CNN
+F 0 "#PWR3" H 1600 4240 20  0001 C CNN
 F 1 "+5V" H 1600 4240 30  0000 C CNN
 F 2 "" H 1600 4150 60  0001 C CNN
@@
 $EndComp
 $Comp
-L GND #PWR016
+L GND #PWR4
 U 1 1 583F4DAA
 P 1600 4650
-F 0 "#PWR016" H 1600 4650 30  0001 C CNN
+F 0 "#PWR4" H 1600 4650 30  0001 C CNN
 F 1 "GND" H 1600 4580 30  0001 C CNN
 F 2 "" H 1600 4650 60  0001 C CNN
@@
 $EndComp
 $Comp
-L GND #PWR017
+L GND #PWR2
 U 1 1 583F4E0C
 P 1600 3650
-F 0 "#PWR017" H 1600 3650 30  0001 C CNN
+F 0 "#PWR2" H 1600 3650 30  0001 C CNN
 F 1 "GND" H 1600 3580 30  0001 C CNN
 F 2 "" H 1600 3650 60  0001 C CNN
@@
 P 9300 4100
 F 0 "D6" H 9250 4000 50  0000 L CNN
-F 1 "1N4002" H 9150 4200 50  0000 L CNN
+F 1 "1N4007" H 9150 4200 50  0000 L CNN
 F 2 "Diodes_ThroughHole:Diode_DO-41_SOD81_Horizontal_RM10" V 9300 4100 60  0001 C CNN
 F 3 "" V 9300 4100 60  0000 C CNN
@@
 P 9300 1850
 F 0 "D5" H 9250 1750 50  0000 L CNN
-F 1 "1N4002" H 9150 1950 50  0000 L CNN
+F 1 "1N4007" H 9150 1950 50  0000 L CNN
 F 2 "Diodes_ThroughHole:Diode_DO-41_SOD81_Horizontal_RM10" V 9300 1850 60  0001 C CNN
 F 3 "" V 9300 1850 60  0000 C CNN
@@
 Text Label 10250 3750 0    24   ~ 0
 B_NO
+$Comp
+L R R5
+U 1 1 5841304F
+P 7650 4200
+F 0 "R5" V 7730 4200 50  0000 C CNN
+F 1 "1kΩ" V 7650 4200 50  0000 C CNN
+F 2 "Resistors_ThroughHole:Resistor_Horizontal_RM10mm" V 7580 4200 30  0001 C CNN
+F 3 "" H 7650 4200 30  0000 C CNN
+	1    7650 4200
+	0    1    1    0
+$EndComp
+Wire Wire Line
+	7350 4200 7500 4200
+$Comp
+L R R4
+U 1 1 58414D97
+P 7650 1950
+F 0 "R4" V 7730 1950 50  0000 C CNN
+F 1 "1kΩ" V 7650 1950 50  0000 C CNN
+F 2 "Resistors_ThroughHole:Resistor_Horizontal_RM10mm" V 7580 1950 30  0001 C CNN
+F 3 "" H 7650 1950 30  0000 C CNN
+	1    7650 1950
+	0    1    1    0
+$EndComp
+Wire Wire Line
+	7350 1950 7500 1950
 $EndSCHEMATC

Commit message: Garage Assistant: Updating
Parts:
- added C3: 100µF, Capacitors_ThroughHole:CP_Radial_D6.3mm_P2.50mm, symbol CP_Small
- added D8: LED_OPT, LEDs:LED_D3.0mm, symbol LED
- added R7: 220Ω, Resistors_ThroughHole:Resistor_Horizontal_RM7mm, symbol R
- D10: renamed from D9; value LED_B -> B
- D5: renamed from D7; footprint LEDs:LED-5MM -> LEDs:LED_D5.0mm
- D9: renamed from D8; value LED_A -> A
- renumbered D5 to D6, D6 to D7, R6 to R4, R4 to R5, R5 to R6, R7 to R8, R8 to R9
Connections:
- net +5VDC is gone; now on net +5V: D6.1 (K), D7.1 (K), RLY1.2, RLY2.2
- net +5V: now also C3.1
- net GND: now also C3.2, D8.1 (K)
- net OPT_LED: now reaches UC1.24 (D13/PWM/LED)
- net OPT_LED: now also R7.2
- new net: D8.2 (A), R7.1
- no-connect marks 19 -> 18
Other:
- note added: "Optional LED"
- moved on the sheet: C2, D1, D10, D2, D3, D4, D5, D6, D7, D9, JP1, JP2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
