File: Circuits/Common Slot PSU Card/Common Slot v2/Common Slot v2.sch (KiCad schematic (older format))
At the start: 61 parts, among them J1 32x2P Card Edge, J10 A1, J11 A2, J12 +12V, J13 0V, J14 +12V, J15 +12V, J16 +12V, J17 0V, J18 0V, J19 0V, J2 ENj, J20 +12V, J21 +12V, J22 +12V, J23 +12V, J24 0V, J25 0V, J26 0V, J27 0V, J28 +12V, J29 +12V, J3 ENi, J30 +12V, J31 +12V, J32 0V, J33 0V, J34 0V, J35 0V, J36 +12V, J37 +12V, J38 +12V, J39 0V, J4 µMolex, J40 0V, J41 0V, J42 +12V, J43 +12V, J44 0V, J45 0V, J46 Isense, J47 Status, J5 5Vsb, J6 12Vsb, J7 Vdisplay, J8 I2C, J9 A0, SW1 ENsw, U1 LTV-817, U2 L7805

Commit message: Common Slot: Added v2 (Mounting hole variant)
Parts:
- J47: footprint Footprints:WIRE-16AWG -> Footprints:WIRE-20AWG
Changed lines of the file:
@@
 EESchema Schematic File Version 4
-LIBS:Common Slot v1-cache
+LIBS:Common Slot v2-cache
 EELAYER 30 0
 EELAYER END
@@
 F 0 "J47" H 8980 4142 50  0000 L CNN
 F 1 "Status" H 8980 4051 50  0000 L CNN
-F 2 "Footprints:WIRE-16AWG" H 8900 4100 50  0001 C CNN
+F 2 "Footprints:WIRE-20AWG" H 8900 4100 50  0001 C CNN
 F 3 "~" H 8900 4100 50  0001 C CNN
 	1    8900 4100
