File: Circuits/SerialGPS/SerialGPS.kicad_pcb (KiCad board)
At the start: 2 copper layers, 73.7 x 48.9 mm, 57 parts, among them IC1 MAX3232, IC2 EEPROM, J1 ANT, P1 USB, P2 AT, P3 DTK, P4 PWR, P5 TP, Q1 2N2222, U1 LM1117-3.3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

Commit message: SerialGPS: Added documentation
Parts:
- removed the ? at (115.8, 79.0)
- moved ? 0.10 mm to (114.4, 105.9)
Routing:
- net RS232_RX: track 24.4 -> 26.4 mm
Other:
- board text added: "+4.5V-20V"
- board text added: "v1.1"
- board text removed: "+5V"
- board text removed: "v1.0"
Changed lines of the file:
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@@
 (kicad_pcb (version 4) (host pcbnew 4.0.4-stable)
   (general
-    (links 110)
+    (links 109)
     (no_connects 0)
     (area 42.54 56.15 133.154075 115.590265)
     (thickness 1.6)
     (drawings 75)
-    (tracks 335)
+    (tracks 336)
     (zones 0)
-    (modules 57)
+    (modules 56)
     (nets 60)
   )
@@
   )
   (module Parts:VIA-0.6mm (layer F.Cu)
-    (at 114.427 105.791)
-    (fp_text reference "" (at 0 1.27) (layer F.SilkS) hide
-      (effects (font (size 1 1) (thickness 0.15)))
-    )
-    (fp_text value "" (at 0 -1.27) (layer F.Fab) hide
-      (effects (font (size 1 1) (thickness 0.15)))
-    )
-    (pad 1 thru_hole circle (at 0 0) (size 0.6 0.6) (drill 0.3) (layers *.Cu)
-      (net 1 GND) (zone_connect 2))
-  )
-  (module Parts:VIA-0.6mm (layer F.Cu)
-    (at 115.824 78.994)
+    (at 114.427 105.8926)
     (fp_text reference "" (at 0 1.27) (layer F.SilkS) hide
       (effects (font (size 1 1) (thickness 0.15)))
@@
     (at 53.975 103.505 180)
     (attr smd)
-    (fp_text reference J1 (at -1.905 2.54 180) (layer F.SilkS) hide
+    (fp_text reference J1 (at -2.3368 2.794 180) (layer F.Fab)
       (effects (font (size 0.762 0.762) (thickness 0.1524)))
     )
-    (fp_text value ANT (at -3.175 -1.905 180) (layer F.SilkS)
+    (fp_text value ANT (at 0 2.9464 180) (layer F.SilkS)
       (effects (font (size 0.762 0.762) (thickness 0.1524)))
     )
@@
     (tags "capacitor 1206")
     (attr smd)
-    (fp_text reference C9 (at -2.032 -1.905) (layer F.SilkS)
+    (fp_text reference C9 (at 6.8326 8.9408) (layer F.SilkS)
       (effects (font (size 1 1) (thickness 0.15)))
     )
@@
     (tags "LED 0603")
     (attr smd)
-    (fp_text reference D2 (at 0 -1.45) (layer F.SilkS)
+    (fp_text reference D2 (at 0 -1.524) (layer F.SilkS)
       (effects (font (size 1 1) (thickness 0.15)))
     )
@@
     (tags "LED 0603")
     (attr smd)
-    (fp_text reference D3 (at 0 -1.45) (layer F.SilkS)
+    (fp_text reference D3 (at 0 -1.4986) (layer F.SilkS)
       (effects (font (size 1 1) (thickness 0.15)))
     )
@@
     (tags "LED 0603")
     (attr smd)
-    (fp_text reference D5 (at 0 -1.45) (layer F.SilkS)
+    (fp_text reference D5 (at 0 -1.524) (layer F.SilkS)
       (effects (font (size 1 1) (thickness 0.15)))
     )
@@
     (tags "LED 0603")
     (attr smd)
-    (fp_text reference D6 (at 0 -1.45 180) (layer F.SilkS)
+    (fp_text reference D6 (at 0 1.4986 180) (layer F.SilkS)
       (effects (font (size 1 1) (thickness 0.15)))
     )
@@
     (effects (font (size 0.8 0.8) (thickness 0.15)))
   )
-  (gr_text v1.0 (at 111.76 58.928) (layer F.SilkS)
+  (gr_text v1.1 (at 111.76 58.928) (layer F.SilkS)
     (effects (font (size 1 1) (thickness 0.2)))
   )
@@
     (effects (font (size 0.7 0.7) (thickness 0.15)) (justify left))
   )
-  (gr_text "E  B  C" (at 67.818 96.901) (layer F.SilkS)
+  (gr_text "E  B  C" (at 67.7164 96.9264) (layer F.SilkS)
     (effects (font (size 1 1) (thickness 0.15)))
   )
@@
     (effects (font (size 0.6 0.6) (thickness 0.15)))
   )
-  (gr_text +5V (at 55.245 58.42 180) (layer F.SilkS)
+  (gr_text +4.5V-20V (at 53.975 58.4454 180) (layer F.SilkS)
     (effects (font (size 0.6 0.6) (thickness 0.15)))
   )
@@
   (segment (start 62.639 79.784) (end 62.639 81.255) (width 1) (layer F.Cu) (net 3))
   (segment (start 58.932478 69.337522) (end 59.055 69.215) (width 1) (layer F.Cu) (net 3))
+  (segment (start 64.135 85.725) (end 60.071 85.725) (width 1) (layer F.Cu) (net 4))
+  (segment (start 60.339 83.8314) (end 60.071 84.0994) (width 1) (layer F.Cu) (net 4))
+  (segment (start 60.071 84.0994) (end 60.071 85.725) (width 1) (layer F.Cu) (net 4))
+  (segment (start 60.339 81.255) (end 60.339 83.8314) (width 1) (layer F.Cu) (net 4))
   (segment (start 97.028 62.611) (end 97.79 63.373) (width 1) (layer F.Cu) (net 4))
   (segment (start 97.79 63.373) (end 97.79 64.262) (width 1) (layer F.Cu) (net 4))
@@
   (segment (start 64.135 85.725) (end 66.421 83.439) (width 1) (layer F.Cu) (net 4))
   (segment (start 69.342 75.692) (end 75.565 81.915) (width 1) (layer F.Cu) (net 4))
-  (segment (start 60.339 81.255) (end 60.339 85.457) (width 1) (layer F.Cu) (net 4))
-  (segment (start 60.339 85.457) (end 60.071 85.725) (width 1) (layer F.Cu) (net 4))
   (segment (start 69.342 70.612) (end 69.342 70.739) (width 1) (layer B.Cu) (net 4))
   (segment (start 69.342 70.739) (end 69.342 75.692) (width 1) (layer F.Cu) (net 4))
   (segment (start 60.339 74.955) (end 68.605 74.955) (width 1) (layer F.Cu) (net 4))
   (segment (start 68.605 74.955) (end 69.342 75.692) (width 1) (layer F.Cu) (net 4))
-  (segment (start 59.69 85.725) (end 63.881 85.725) (width 1) (layer F.Cu) (net 4))
   (segment (start 94.161 64.697) (end 96.107001 64.697) (width 0.69) (layer F.Cu) (net 4))
   (segment (start 97.822 74.295) (end 97.822 75.9145) (width 0.25) (layer F.Cu) (net 5))
@@
   (segment (start 97.502 70.197) (end 98.933 71.628) (width 0.25) (layer F.Cu) (net 22))
   (segment (start 94.161 70.197) (end 97.502 70.197) (width 0.25) (layer F.Cu) (net 22))
-  (segment (start 59.845 103.505) (end 59.845 105.005) (width 0.25) (layer F.Cu) (net 23))
-  (segment (start 59.845 105.005) (end 60.670001 105.830001) (width 0.25) (layer F.Cu) (net 23))
-  (segment (start 60.670001 105.830001) (end 68.794999 105.830001) (width 0.25) (layer F.Cu) (net 23))
-  (segment (start 68.794999 105.830001) (end 71.635009 102.989991) (width 0.25) (layer F.Cu) (net 23))
+  (segment (start 59.845 103.505) (end 59.845 105.0316) (width 0.25) (layer F.Cu) (net 23))
+  (segment (start 59.845 105.0316) (end 60.4774 105.664) (width 0.25) (layer F.Cu) (net 23))
+  (segment (start 60.4774 105.664) (end 68.961 105.664) (width 0.25) (layer F.Cu) (net 23))
+  (segment (start 68.961 105.664) (end 71.635009 102.989991) (width 0.25) (layer F.Cu) (net 23))
   (segment (start 71.635009 102.989991) (end 77.858599 102.989991) (width 0.25) (layer F.Cu) (net 23))
   (segment (start 77.858599 102.989991) (end 84.836 96.01259) (width 0.25) (layer F.Cu) (net 23))
@@
   (segment (start 97.028 97.409) (end 97.028 95.762) (width 0.25) (layer F.Cu) (net 58))
   (segment (start 98.425 95.25) (end 97.54 95.25) (width 0.25) (layer F.Cu) (net 58))
+  (segment (start 115.6462 73.025) (end 113.665 73.025) (width 0.25) (layer B.Cu) (net 59))
+  (segment (start 113.665 73.025) (end 112.395 71.755) (width 0.25) (layer B.Cu) (net 59))
+  (segment (start 116.84 74.2188) (end 115.6462 73.025) (width 0.25) (layer B.Cu) (net 59))
+  (segment (start 116.84 82.3976) (end 116.84 74.2188) (width 0.25) (layer B.Cu) (net 59))
+  (segment (start 116.078 83.1596) (end 116.84 82.3976) (width 0.25) (layer B.Cu) (net 59))
+  (segment (start 113.6904 83.1596) (end 116.078 83.1596) (width 0.25) (layer B.Cu) (net 59))
+  (segment (start 112.395 84.455) (end 113.6904 83.1596) (width 0.25) (layer B.Cu) (net 59))
   (segment (start 109.855 84.455) (end 112.395 84.455) (width 0.25) (layer F.Cu) (net 59))
-  (segment (start 112.395 84.455) (end 113.665 83.185) (width 0.25) (layer F.Cu) (net 59))
-  (segment (start 113.665 83.185) (end 115.57 83.185) (width 0.25) (layer F.Cu) (net 59))
-  (segment (start 115.57 83.185) (end 116.205 82.55) (width 0.25) (layer F.Cu) (net 59))
-  (segment (start 116.205 82.55) (end 116.205 80.645) (width 0.25) (layer F.Cu) (net 59))
-  (segment (start 116.205 80.645) (end 113.665 78.105) (width 0.25) (layer F.Cu) (net 59))
-  (segment (start 113.665 78.105) (end 113.665 73.025) (width 0.25) (layer F.Cu) (net 59))
-  (segment (start 113.665 73.025) (end 112.395 71.755) (width 0.25) (layer F.Cu) (net 59))
   (segment (start 109.22 83.82) (end 109.855 84.455) (width 0.25) (layer F.Cu) (net 59))
   (segment (start 109.22 83.185) (end 109.22 83.82) (width 0.25) (layer F.Cu) (net 59))

Commit message: Working on Serial GPS
Other:
- net class Default removed
- net class Neo removed
- net class Power removed
