File: Circuits/ESPSauna/ESPSauna.kicad_pcb (KiCad board)
At the start: 2 copper layers, 68.5 x 62 mm, 44 parts, among them J1 AudioJack3, J2 Conn_01x04, Q1 AO3400A, Q2 AO3400A, U1 AP63203WU, U3 AM2302, U4 ESP32-DEVKIT-V1

Commit message: Overhaul of html pages; pulling out js and css into separate files, using no image fallback, adding espprobe, espdrive and espradiator stubs awaiting images
Parts:
- added C11: 10μF, Capacitor_SMD:C_1206_3216Metric_Pad1.33x1.80mm_HandSolder, B.Cu at (147.0, 105.0)
- added R9: 43kΩ, Resistor_THT:R_Axial_DIN0207_L6.3mm_D2.5mm_P10.16mm_Horizontal, F.Cu at (157.7, 79.9)
- C10: value 33nF -> 1μF
- J1: value AudioJack3 -> CT Clamp
- J2: value Conn_01x04 -> SHT45
- moved R6 26.4 mm to (153.0, 99.0), turned to 0 degrees
- moved R4 18.6 mm to (148.0, 99.0), turned to 0 degrees
- moved U3 1.98 mm to (151.6, 73.4)
- moved R1 1.87 mm to (148.9, 72.1)
- moved J2 1.40 mm to (156.0, 66.1)
- moved C10 1.00 mm to (128.0, 84.0), turned to -90 degrees
- moved J1 0.40 mm to (155.0, 88.4)
- renumbered C5 to C1, C6 to C2, C1 to C3, C2 to C4, C3 to C5, C4 to C6
Connections:
- C10 pad 1: Net-(C10-Pad1) -> Sense
- J1 pad R: GNDREF -> unconnected-(J1-PadR)
- J1 pad S: GNDREF -> Net-(C11-Pad1)
- J1 pad T: Net-(C10-Pad1) -> Net-(J1-PadT)
- R4 pad 2: Net-(C10-Pad1) -> Net-(C11-Pad1)
- R5 pad 2: Net-(C10-Pad1) -> Net-(J1-PadT)
- R6 pad 1: Net-(C10-Pad1) -> Net-(C11-Pad1)
Routing:
- net Net-(C11-Pad1): track 0.00 -> 31.8 mm
- net Net-(C10-Pad1): track 28.9 -> 0.00 mm
- net Net-(J1-PadT): track 0.00 -> 22.7 mm
- net +3V3: track 109.0 -> 104.3 mm
- net Sense: track 16.8 -> 19.7 mm
- net AC1: track 36.2 -> 34.4 mm
- net DHT: track 25.9 -> 24.4 mm
- net SCL: track 25.8 -> 27.2 mm
- net SDA: track 18.4 -> 19.8 mm
- added copper zone on B.Cu, net Net-(J1-PadT)
- removed copper zone on B.Cu, net Net-(C10-Pad1)
Other:
- outline, holes or cut-outs redrawn
- board text added: "2026.06.18"
- board text added: "ESPSauna v1.1"
- board text added: "ehryk.github.io/espsauna"
- board text removed: "DHT22 / AM2302"
- board text removed: "ESPSauna v1.0 2026.05.24"
