File: Circuits/ESPDrive/ESPDrive.kicad_pcb (KiCad board)
At the start: 4 copper layers, 44 x 64 mm, 58 parts, among them Q2 AO3401A, Q3 AO3400A, U1 AP63203WU, U2 AP63201WU, U3 LTV-827S

Commit message: Added ESP images; added sections to index.html
Other:
- board text added: "ehryk.github.io/espdrive"
