File: Circuits/ESPRadiator/ESPRadiator.kicad_pcb (KiCad board)
At the start: 2 copper layers, 50 x 57 mm, 49 parts, among them Q1 AO3401A, Q2 MMBT3904, Q3 IRLZ44N, Q4 IRLZ44N, U1 AP63203WU, U2 LTV-827S

Commit message: Added ESP images; added sections to index.html
Other:
- board text added: "ESPRadiator v1.0"
- board text removed: "ESPFan v1.0"
