File: Circuits/ESPFridge/ESPFridge.kicad_pcb (KiCad board)
At the start: 2 copper layers, 21.2 x 77.6 mm, 30 parts, among them J1 Conn_01x06_Socket, Q1 AO3401A, Q2 MMBT3904, U1 ESP32-C3-WROOM-02, U2 DW01A, U3 8205A, U4 OPT3001DNPRQ1, U5 MCP1700x-330xxTT, U6 TMP117xxDRV

Commit message: Overhaul of html pages; pulling out js and css into separate files, using no image fallback, adding espprobe, espdrive and espradiator stubs awaiting images
Other:
- board text added: "ehryk.github.io/espfridge"

Commit message: ESPFridge Fab layer and bom updates
Other:
- board text added: "(1206)"
- board text added: "(1210)"
- board text added: "U3"
- board text added: "U4"
